Commit message: Add rear wheels and joint state GUI to rover model

File: src/rover_description/urdf/rover.urdf.xacro (robot description, xacro)
@@ -9,4 +9,7 @@
   <xacro:property name="wheel_radius" value="0.15875"/>
   <xacro:property name="ground_clearance" value="0.08"/>
+  <xacro:property name="track_width" value="0.559"/>
+  <xacro:property name="wheel_width" value="0.1016"/>
+  <xacro:property name="wheel_mass" value="1.5"/>
   <!-- Height of the chassis box center, measured from base_link -->
   <xacro:property name="chassis_z"
@@ -14,4 +17,7 @@
   <material name="chassis_grey">
     <color rgba="0.5 0.5 0.55 1.0"/>
+  </material>
+  <material name="wheel_black">
+    <color rgba="0.1 0.1 0.1 1.0"/>
   </material>
   <!-- ===== Frames ===== -->
@@ -46,3 +52,37 @@
     </inertial>
   </link>
+    <!-- ===== Wheels ===== -->
+  <xacro:macro name="wheel" params="prefix x y">
+    <link name="${prefix}_wheel">
+      <visual>
+        <origin xyz="0 0 0" rpy="${pi / 2} 0 0"/>
+        <geometry>
+          <cylinder radius="${wheel_radius}" length="${wheel_width}"/>
+        </geometry>
+        <material name="wheel_black"/>
+      </visual>
+      <collision>
+        <origin xyz="0 0 0" rpy="${pi / 2} 0 0"/>
+        <geometry>
+          <cylinder radius="${wheel_radius}" length="${wheel_width}"/>
+        </geometry>
+      </collision>
+      <inertial>
+        <mass value="${wheel_mass}"/>
+        <inertia
+          ixx="${wheel_mass / 12 * (3 * wheel_radius**2 + wheel_width**2)}"
+          iyy="${wheel_mass * wheel_radius**2 / 2}"
+          izz="${wheel_mass / 12 * (3 * wheel_radius**2 + wheel_width**2)}"
+          ixy="0" ixz="0" iyz="0"/>
+      </inertial>
+    </link>
+    <joint name="${prefix}_wheel_joint" type="continuous">
+      <parent link="base_link"/>
+      <child link="${prefix}_wheel"/>
+      <origin xyz="${x} ${y} 0" rpy="0 0 0"/>
+      <axis xyz="0 1 0"/>
+    </joint>
+  </xacro:macro>
+  <xacro:wheel prefix="rear_left" x="0" y="${track_width / 2}"/>
+  <xacro:wheel prefix="rear_right" x="0" y="${-track_width / 2}"/>
 </robot>

Commit message: Add steerable front wheels to rover model

File: src/rover_description/urdf/rover.urdf.xacro (robot description, xacro)
@@ -12,4 +12,5 @@
   <xacro:property name="wheel_width" value="0.1016"/>
   <xacro:property name="wheel_mass" value="1.5"/>
+  <xacro:property name="max_steer_angle" value="0.7"/>
   <!-- Height of the chassis box center, measured from base_link -->
   <xacro:property name="chassis_z"
@@ -53,5 +54,5 @@
   </link>
     <!-- ===== Wheels ===== -->
-  <xacro:macro name="wheel" params="prefix x y">
+  <xacro:macro name="wheel" params="prefix parent x y">
     <link name="${prefix}_wheel">
       <visual>
@@ -78,5 +79,5 @@
     </link>
     <joint name="${prefix}_wheel_joint" type="continuous">
-      <parent link="base_link"/>
+      <parent link="${parent}"/>
       <child link="${prefix}_wheel"/>
       <origin xyz="${x} ${y} 0" rpy="0 0 0"/>
@@ -84,5 +85,24 @@
     </joint>
   </xacro:macro>
-  <xacro:wheel prefix="rear_left" x="0" y="${track_width / 2}"/>
-  <xacro:wheel prefix="rear_right" x="0" y="${-track_width / 2}"/>
+  <xacro:macro name="steering_knuckle" params="prefix y">
+    <link name="${prefix}_knuckle">
+      <inertial>
+        <mass value="0.5"/>
+        <inertia ixx="0.001" iyy="0.001" izz="0.001" ixy="0" ixz="0" iyz="0"/>
+      </inertial>
+    </link>
+    <joint name="${prefix}_steer_joint" type="revolute">
+      <parent link="base_link"/>
+      <child link="${prefix}_knuckle"/>
+      <origin xyz="${wheelbase} ${y} 0" rpy="0 0 0"/>
+      <axis xyz="0 0 1"/>
+      <limit lower="${-max_steer_angle}" upper="${max_steer_angle}"
+             effort="50" velocity="2.0"/>
+    </joint>
+    <xacro:wheel prefix="${prefix}" parent="${prefix}_knuckle" x="0" y="0"/>
+  </xacro:macro>
+  <xacro:wheel prefix="rear_left" parent="base_link" x="0" y="${track_width / 2}"/>
+  <xacro:wheel prefix="rear_right" parent="base_link" x="0" y="${-track_width / 2}"/>
+  <xacro:steering_knuckle prefix="front_left" y="${track_width / 2}"/>
+  <xacro:steering_knuckle prefix="front_right" y="${-track_width / 2}"/>
 </robot>

Commit message: Add scissor lift with prismatic joint carrying the LIDAR

File: src/rover_description/urdf/rover.urdf.xacro (robot description, xacro)
@@ -16,4 +16,20 @@
   <xacro:property name="chassis_z"
                   value="${ground_clearance + chassis_height / 2 - wheel_radius}"/>
+  <!-- Top surface of the chassis, measured from base_link -->
+  <xacro:property name="chassis_top_z"
+                  value="${ground_clearance + chassis_height - wheel_radius}"/>
+  <!-- Sensor positions in meters from base_link (rear axle center, x forward, z up) -->
+  <!-- Scissor lift: platform slides straight up from the chassis top -->
+  <xacro:property name="lift_x" value="${wheelbase / 2}"/>
+  <xacro:property name="lift_y" value="0.0"/>
+  <xacro:property name="lift_travel" value="1.2192"/>
+  <xacro:property name="lift_platform_mass" value="5.0"/>
+  <xacro:property name="lidar_offset" value="0.03"/>
+  <xacro:property name="imu_x" value="${wheelbase / 2}"/>
+  <xacro:property name="imu_y" value="0.0"/>
+  <xacro:property name="imu_z" value="${chassis_z}"/>
+  <xacro:property name="gps_x" value="0.0"/>
+  <xacro:property name="gps_y" value="0.0"/>
+  <xacro:property name="gps_z" value="${chassis_top_z + 0.03}"/>
   <material name="chassis_grey">
     <color rgba="0.5 0.5 0.55 1.0"/>
@@ -21,4 +37,7 @@
   <material name="wheel_black">
     <color rgba="0.1 0.1 0.1 1.0"/>
+  </material>
+  <material name="sensor_blue">
+    <color rgba="0.1 0.3 0.8 1.0"/>
   </material>
   <!-- ===== Frames ===== -->
@@ -106,3 +125,69 @@
   <xacro:steering_knuckle prefix="front_left" y="${track_width / 2}"/>
   <xacro:steering_knuckle prefix="front_right" y="${-track_width / 2}"/>
+  <!-- ===== Sensors ===== -->
+  <!-- Lift platform: slides up and down on a prismatic joint -->
+  <link name="lift_platform">
+    <visual>
+      <geometry>
+        <box size="0.4 0.4 0.02"/>
+      </geometry>
+      <material name="chassis_grey"/>
+    </visual>
+    <collision>
+      <geometry>
+        <box size="0.4 0.4 0.02"/>
+      </geometry>
+    </collision>
+    <inertial>
+      <mass value="${lift_platform_mass}"/>
+      <inertia ixx="0.067" iyy="0.067" izz="0.133" ixy="0" ixz="0" iyz="0"/>
+    </inertial>
+  </link>
+  <joint name="lift_joint" type="prismatic">
+    <parent link="base_link"/>
+    <child link="lift_platform"/>
+    <origin xyz="${lift_x} ${lift_y} ${chassis_top_z}" rpy="0 0 0"/>
+    <axis xyz="0 0 1"/>
+    <limit lower="0.0" upper="${lift_travel}" effort="500" velocity="0.05"/>
+  </joint>
+  <!-- LIDAR rides on the platform -->
+  <link name="lidar_link">
+    <visual>
+      <geometry>
+        <cylinder radius="0.04" length="0.04"/>
+      </geometry>
+      <material name="sensor_blue"/>
+    </visual>
+  </link>
+  <joint name="lidar_joint" type="fixed">
+    <parent link="lift_platform"/>
+    <child link="lidar_link"/>
+    <origin xyz="0 0 ${lidar_offset}" rpy="0 0 0"/>
+  </joint>
+  <link name="imu_link">
+    <visual>
+      <geometry>
+        <box size="0.04 0.04 0.02"/>
+      </geometry>
+      <material name="sensor_blue"/>
+    </visual>
+  </link>
+  <joint name="imu_joint" type="fixed">
+    <parent link="base_link"/>
+    <child link="imu_link"/>
+    <origin xyz="${imu_x} ${imu_y} ${imu_z}" rpy="0 0 0"/>
+  </joint>
+  <link name="gps_link">
+    <visual>
+      <geometry>
+        <box size="0.06 0.06 0.02"/>
+      </geometry>
+      <material name="sensor_blue"/>
+    </visual>
+  </link>
+  <joint name="gps_joint" type="fixed">
+    <parent link="base_link"/>
+    <child link="gps_link"/>
+    <origin xyz="${gps_x} ${gps_y} ${gps_z}" rpy="0 0 0"/>
+  </joint>
 </robot>

Commit message: Add first tree to the world and raise the sim GPS above the LIDAR plane

File: src/rover_description/urdf/rover.urdf.xacro (robot description, xacro)
@@ -31,5 +31,5 @@
   <xacro:property name="gps_x" value="0.0"/>
   <xacro:property name="gps_y" value="0.0"/>
-  <xacro:property name="gps_z" value="${chassis_top_z + 0.03}"/>
+  <xacro:property name="gps_z" value="${chassis_top_z + 0.15}"/>
   <material name="chassis_grey">
     <color rgba="0.5 0.5 0.55 1.0"/>

Commit message: Add six ultrasonic sensor frames to the rover model

File: src/rover_description/urdf/rover.urdf.xacro (robot description, xacro)
@@ -32,4 +32,10 @@
   <xacro:property name="gps_y" value="0.0"/>
   <xacro:property name="gps_z" value="${chassis_top_z + 0.15}"/>
+    <!-- Ultrasonics: PLACEHOLDER positions. z is 3 in above the top of the wheels -->
+  <xacro:property name="us_z" value="${wheel_radius + 0.0762}"/>
+  <xacro:property name="us_front_x" value="${wheelbase / 2 + chassis_length / 2 + 0.01}"/>
+  <xacro:property name="us_rear_x" value="${wheelbase / 2 - chassis_length / 2 - 0.01}"/>
+  <xacro:property name="us_side_y" value="0.15"/>
+  <xacro:property name="us_angle" value="0.26"/>
   <material name="chassis_grey">
     <color rgba="0.5 0.5 0.55 1.0"/>
@@ -192,3 +198,28 @@
   </joint>
   <xacro:include filename="$(find rover_description)/urdf/rover.gazebo.xacro"/>
+  <!-- ===== Ultrasonic sensors ===== -->
+  <material name="us_green">
+    <color rgba="0.1 0.6 0.2 1.0"/>
+  </material>
+  <xacro:macro name="ultrasonic" params="id x y yaw">
+    <link name="us_${id}">
+      <visual>
+        <geometry>
+          <box size="0.02 0.045 0.02"/>
+        </geometry>
+        <material name="us_green"/>
+      </visual>
+    </link>
+    <joint name="us_${id}_joint" type="fixed">
+      <parent link="base_link"/>
+      <child link="us_${id}"/>
+      <origin xyz="${x} ${y} ${us_z}" rpy="0 0 ${yaw}"/>
+    </joint>
+  </xacro:macro>
+  <xacro:ultrasonic id="front_left" x="${us_front_x}" y="${us_side_y}" yaw="${us_angle}"/>
+  <xacro:ultrasonic id="front_mid" x="${us_front_x}" y="0" yaw="0"/>
+  <xacro:ultrasonic id="front_right" x="${us_front_x}" y="${-us_side_y}" yaw="${-us_angle}"/>
+  <xacro:ultrasonic id="rear_left" x="${us_rear_x}" y="${us_side_y}" yaw="${pi - us_angle}"/>
+  <xacro:ultrasonic id="rear_mid" x="${us_rear_x}" y="0" yaw="${pi}"/>
+  <xacro:ultrasonic id="rear_right" x="${us_rear_x}" y="${-us_side_y}" yaw="${pi + us_angle}"/>
 </robot>

Commit message: Lower the sim GPS onto the chassis, just under the LIDAR plane

File: src/rover_description/urdf/rover.urdf.xacro (robot description, xacro)
@@ -31,5 +31,5 @@
   <xacro:property name="gps_x" value="0.0"/>
   <xacro:property name="gps_y" value="0.0"/>
-  <xacro:property name="gps_z" value="${chassis_top_z + 0.15}"/>
+  <xacro:property name="gps_z" value="${chassis_top_z + 0.01}"/>
     <!-- Ultrasonics: PLACEHOLDER positions. z is 3 in above the top of the wheels -->
   <xacro:property name="us_z" value="${wheel_radius + 0.0762}"/>
